File: keyboard_test.kicad_pcb (KiCad board)
At the start: 2 copper layers, 62.7 x 38.1 mm, 24 parts, among them SW1 SW_Push, U1 ATmega32U4-AU, Y1 Crystal_GND24_Small

Commit message: Fixed errors
-Fixed silkscreen error (swapped R1 and C7)
-Fixed crystal connections & adjusted routing
-Put gerbers in their own folder
Parts:
- moved C5 0.89 mm to (39.1, 77.6), turned to 270 degrees
- moved C6 0.89 mm to (30.5, 77.6), turned to 90 degrees
- moved Y1 0.89 mm to (34.8, 77.6)
Connections:
- Y1 pad 1: GND -> Net-(C5-Pad1)
- Y1 pad 2: Net-(C6-Pad1) -> GND
- Y1 pad 3: GND -> Net-(C6-Pad1)
- Y1 pad 4: Net-(C5-Pad1) -> GND
Routing:
- net GND: track 30.8 -> 53.3 mm, vias 12 -> 11
- net Net-(C6-Pad1): track 5.77 -> 11.3 mm
- net Net-(C5-Pad1): track 8.48 -> 7.21 mm
Other:
- board text added: "Rev.2"
- board text removed: "Rev.1"
