File: keyboard_test.sch (KiCad schematic (older format))
At the start: 24 parts, among them SW1 SW_Push, U1 ATmega32U4-AU, Y1 Crystal_GND24_Small

Commit message: Layout & routing complete
Connections:
- net COL_0: now also U1.29 (PB5)
- net COL_1: now also U1.28 (PB4)
- net GND: now also R4.2; no longer R1.1, R4.1
- net ROW_0: now also U1.30 (PB6)
- net ROW_1: now also U1.27 (PD7)
- net at SW1.2, U1.13 (~RESET): now also R1.1
- net at U1.33 (~HWB~/PE2): now also R4.1; no longer R4.2
Other:
- moved on the sheet: C5, C6, R1, SW1
Changed lines of the file:
@@
 F 3 "~" H 4600 4950 50  0001 C CNN
 	1    4600 4950
-	0    1    1    0
+	0    -1   -1   0
 $EndComp
 $Comp
@@
 L Device:C_Small C6
 U 1 1 5F981CFB
-P 2500 3300
-F 0 "C6" V 2400 3250 50  0000 L CNN
-F 1 "22p" V 2600 3250 50  0000 L CNN
-F 2 "Capacitor_SMD:C_1206_3216Metric" H 2500 3300 50  0001 C CNN
-F 3 "~" H 2500 3300 50  0001 C CNN
-	1    2500 3300
+P 2550 3300
+F 0 "C6" V 2450 3250 50  0000 L CNN
+F 1 "22p" V 2650 3250 50  0000 L CNN
+F 2 "Capacitor_SMD:C_1206_3216Metric" H 2550 3300 50  0001 C CNN
+F 3 "~" H 2550 3300 50  0001 C CNN
+	1    2550 3300
 	0    1    1    0
 $EndComp
@@
 L Device:C_Small C5
 U 1 1 5F983877
-P 2500 3000
-F 0 "C5" V 2400 2950 50  0000 L CNN
-F 1 "22p" V 2600 2950 50  0000 L CNN
-F 2 "Capacitor_SMD:C_1206_3216Metric" H 2500 3000 50  0001 C CNN
-F 3 "~" H 2500 3000 50  0001 C CNN
-	1    2500 3000
+P 2550 3000
+F 0 "C5" V 2450 2950 50  0000 L CNN
+F 1 "22p" V 2650 2950 50  0000 L CNN
+F 2 "Capacitor_SMD:C_1206_3216Metric" H 2550 3000 50  0001 C CNN
+F 3 "~" H 2550 3000 50  0001 C CNN
+	1    2550 3000
 	0    1    1    0
 $EndComp
 Wire Wire Line
-	2850 3300 2600 3300
+	2850 3300 2650 3300
 Connection ~ 2850 3300
 Wire Wire Line
-	2850 3000 2600 3000
+	2850 3000 2650 3000
 Connection ~ 2850 3000
 $Comp
 L power:GND #PWR0109
 U 1 1 5F9865A7
-P 2350 3400
-F 0 "#PWR0109" H 2350 3150 50  0001 C CNN
-F 1 "GND" H 2355 3227 50  0000 C CNN
-F 2 "" H 2350 3400 50  0001 C CNN
-F 3 "" H 2350 3400 50  0001 C CNN
-	1    2350 3400
-	1    0    0    -1
-$EndComp
-Wire Wire Line
-	2350 3400 2350 3300
-Wire Wire Line
-	2350 3300 2400 3300
-Wire Wire Line
-	2350 3300 2350 3000
-Wire Wire Line
-	2350 3000 2400 3000
-Connection ~ 2350 3300
+P 2400 3400
+F 0 "#PWR0109" H 2400 3150 50  0001 C CNN
+F 1 "GND" H 2405 3227 50  0000 C CNN
+F 2 "" H 2400 3400 50  0001 C CNN
+F 3 "" H 2400 3400 50  0001 C CNN
+	1    2400 3400
+	1    0    0    -1
+$EndComp
+Wire Wire Line
+	2400 3400 2400 3300
+Wire Wire Line
+	2400 3300 2450 3300
+Wire Wire Line
+	2400 3300 2400 3000
+Wire Wire Line
+	2400 3000 2450 3000
+Connection ~ 2400 3300
 $Comp
 L Switch:SW_Push SW1
 U 1 1 5F98A16A
-P 2900 2850
-F 0 "SW1" H 2900 3135 50  0000 C CNN
-F 1 "SW_Push" H 2900 3044 50  0000 C CNN
-F 2 "random-keyboard-parts:SKQG-1155865" H 2900 3050 50  0001 C CNN
-F 3 "~" H 2900 3050 50  0001 C CNN
-	1    2900 2850
-	1    0    0    -1
-$EndComp
-Wire Wire Line
-	3150 2850 3100 2850
-$Comp
-L power:GND #PWR0110
-U 1 1 5F98C5BF
-P 2650 3400
-F 0 "#PWR0110" H 2650 3150 50  0001 C CNN
-F 1 "GND" H 2655 3227 50  0000 C CNN
-F 2 "" H 2650 3400 50  0001 C CNN
-F 3 "" H 2650 3400 50  0001 C CNN
-	1    2650 3400
-	1    0    0    -1
-$EndComp
-Wire Wire Line
-	2650 3400 2650 2850
-Wire Wire Line
-	2650 2850 2700 2850
+P 2650 2850
+F 0 "SW1" H 2650 3135 50  0000 C CNN
+F 1 "SW_Push" H 2650 3044 50  0000 C CNN
+F 2 "random-keyboard-parts:SKQG-1155865" H 2650 3050 50  0001 C CNN
+F 3 "~" H 2650 3050 50  0001 C CNN
+	1    2650 2850
+	1    0    0    -1
+$EndComp
 $Comp
 L Device:R_Small_US R1
 U 1 1 5F99FD61
-P 2650 2700
-F 0 "R1" H 2582 2654 50  0000 R CNN
-F 1 "10k" H 2582 2745 50  0000 R CNN
-F 2 "Resistor_SMD:R_1206_3216Metric" H 2650 2700 50  0001 C CNN
-F 3 "~" H 2650 2700 50  0001 C CNN
-	1    2650 2700
-	1    0    0    1
+P 2900 2700
+F 0 "R1" H 2832 2654 50  0000 R CNN
+F 1 "10k" H 2832 2745 50  0000 R CNN
+F 2 "Resistor_SMD:R_1206_3216Metric" H 2900 2700 50  0001 C CNN
+F 3 "~" H 2900 2700 50  0001 C CNN
+	1    2900 2700
+	-1   0    0    1
 $EndComp
 $Comp
 L power:+5V #PWR0111
 U 1 1 5F9A4780
-P 2650 2550
-F 0 "#PWR0111" H 2650 2400 50  0001 C CNN
-F 1 "+5V" H 2665 2723 50  0000 C CNN
-F 2 "" H 2650 2550 50  0001 C CNN
-F 3 "" H 2650 2550 50  0001 C CNN
-	1    2650 2550
-	1    0    0    -1
-$EndComp
-Wire Wire Line
-	2650 2850 2650 2800
-Connection ~ 2650 2850
-Wire Wire Line
-	2650 2600 2650 2550
+P 2900 2550
+F 0 "#PWR0111" H 2900 2400 50  0001 C CNN
+F 1 "+5V" H 2915 2723 50  0000 C CNN
+F 2 "" H 2900 2550 50  0001 C CNN
+F 3 "" H 2900 2550 50  0001 C CNN
+	1    2900 2550
+	1    0    0    -1
+$EndComp
+Wire Wire Line
+	2900 2850 2900 2800
+Wire Wire Line
+	2900 2600 2900 2550
 Text GLabel 2850 3850 0    50   Input ~ 0
 D+
@@
 Text GLabel 6400 4300 0    50   Input ~ 0
 ROW_1
+Wire Wire Line
+	2850 2850 2900 2850
+Connection ~ 2900 2850
+Wire Wire Line
+	2900 2850 3150 2850
+Wire Wire Line
+	2450 2850 2400 2850
+Wire Wire Line
+	2400 2850 2400 3000
+Connection ~ 2400 3000
+Text GLabel 4400 4750 2    50   Input ~ 0
+ROW_1
+Wire Wire Line
+	4400 4750 4350 4750
+Text GLabel 4400 3450 2    50   Input ~ 0
+ROW_0
+Wire Wire Line
+	4400 3450 4350 3450
+Text GLabel 4400 3350 2    50   Input ~ 0
+COL_0
+Wire Wire Line
+	4400 3350 4350 3350
+Text GLabel 4400 3250 2    50   Input ~ 0
+COL_1
+Wire Wire Line
+	4400 3250 4350 3250
 $EndSCHEMATC

Commit message: Fixed errors
-Fixed silkscreen error (swapped R1 and C7)
-Fixed crystal connections & adjusted routing
-Put gerbers in their own folder
Connections:
- net GND: now also Y1.2, Y1.4; no longer Y1.1, Y1.3
- net at C6.1, U1.16 (XTAL2): now also Y1.3; no longer Y1.2
- net at C5.1, U1.17 (XTAL1): now also Y1.1; no longer Y1.4
Other:
- moved on the sheet: C1, C2, C3, C4, D1, D2, D3, D4, F1, MX1, MX2, MX3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
